File: Apple-68k-FujiNet-Rev0/Apple-68k-FujiNet-Rev0.kicad_pcb (KiCad board)
At the start: 2 copper layers, 80.8 x 55.4 mm, 30 parts, among them J1 Apple IDC-20, J2 Logic Analyzer, J3 UART, J4 SWD, P1 ST-TF-003A, SW1 ButtonA, SW2 Safe Reset, U1 Pico, U2 ESP32-DevKitC-VE

Commit message: Remove ground on Pin 7 for Rev0 boards since Jeff may also use these for Apple II development
Parts:
- removed REF**: OSHW-Logo2_9.8x8mm_SilkScreen, Symbol:OSHW-Logo2_9.8x8mm_SilkScreen
- removed REF**: KiCad-Logo2_5mm_SilkScreen, Symbol:KiCad-Logo2_5mm_SilkScreen
Connections:
- J1 pad 7: GND -> unconnected-(J1-Pin_7-Pad7)
