File: Apple-68k-FujiNet-Rev0/Apple-68k-FujiNet-Rev0.kicad_sch (KiCad schematic)
At the start: 26 parts, among them J1 Apple IDC-20, J2 Logic Analyzer, J3 UART, J4 SWD, P1 ST-TF-003A, SW1 ButtonA, SW2 Safe Reset, U1 Pico, U2 ESP32-DevKitC-VE

Commit message: Remove ground on Pin 7 for Rev0 boards since Jeff may also use these for Apple II development
Connections:
- net GND: no longer J1.7 (Pin_7)
- no-connect marks 39 -> 40
Changed lines of the file:
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@@
   (junction (at 57.15 158.75) (diameter 0) (color 0 0 0 0)
-  )
-  (junction (at 30.48 41.91) (diameter 0) (color 0 0 0 0)
   )
   (junction (at 30.48 36.83) (diameter 0) (color 0 0 0 0)
@@
   (no_connect (at 57.15 59.69))
   (no_connect (at 147.32 41.275))
+  (no_connect (at 44.45 44.45))
   (no_connect (at 212.09 64.135))
   (no_connect (at 252.73 53.975))
@@
     (stroke (width 0) (type default))
   )
-  (wire (pts (xy 30.48 44.45) (xy 44.45 44.45))
-    (stroke (width 0) (type default))
-  )
   (wire (pts (xy 101.6 118.11) (xy 113.665 118.11))
     (stroke (width 0) (type default))
@@
     (stroke (width 0) (type default))
   )
-  (wire (pts (xy 30.48 41.91) (xy 30.48 44.45))
-    (stroke (width 0) (type default))
-  )
